File: PlacaReceptora.sch (KiCad schematic (older format))
At the start: 18 parts, among them J1 JACK_TRS, J2 PainelSolar, J3 Screw_Terminal_Fonte, SW1 SW_CaboP2_PainelSolar, SW2 SW_OnOff, U1 LM386

Commit message: Feito as pcbs dos circuitos emissor e receptor
Feito os fotolitos da versão V1
Parts:
- removed RV3: R_POT_1K_FiltroParaleloACarga, Potentiometers:Potentiometer_Trimmer_ACP_CA14v_Horizontal_Px15.0mm_Py10.0mm, symbol Device:R_POT_US
- removed SW1: SW_CaboP2_PainelSolar, Connector:SW_7x7_6Pinos, symbol Switch:SW_DPDT_x2
- added SW4: SW_DPDT_x2, Connector:SW_7x7_6Pinos, symbol Switch:SW_DPDT_x2
- C1: value CP_FiltroAC -> CP_22uF_FiltroAC; footprint Capacitors_THT:CP_Radial_D6.3mm_P2.50mm -> Capacitors_THT:CP_Radial_Tantal_D6.0mm_P5.00mm
- C2: footprint Capacitors_THT:CP_Radial_D6.3mm_P2.50mm -> Capacitors_THT:CP_Radial_Tantal_D6.0mm_P5.00mm
- C3: footprint Capacitors_THT:CP_Radial_D8.0mm_P2.50mm -> Capacitors_THT:CP_Radial_Tantal_D6.0mm_P5.00mm
- C4: value CP_0.1nF_Estabilidade -> CP_10uF_Estabilidade; footprint Capacitors_THT:CP_Radial_D7.5mm_P2.50mm -> Capacitors_THT:CP_Radial_Tantal_D6.0mm_P5.00mm
- C5: value CP_FiltroAC_470nF -> CP_FiltroAC_220nF; footprint Capacitors_THT:CP_Radial_D6.3mm_P2.50mm -> Capacitors_THT:CP_Radial_Tantal_D6.0mm_P5.00mm
- C6, C7: footprint Capacitors_THT:CP_Radial_D5.0mm_P2.50mm -> Capacitors_THT:CP_Radial_Tantal_D6.0mm_P5.00mm
- RV1: footprint Potentiometers:Potentiometer_Trimmer_ACP_CA14v_Horizontal_Px15.0mm_Py10.0mm -> Potentiometers:Potentiometer_Piher_PC-16_Single_Vertical
- RV2: footprint Potentiometers:Potentiometer_Trimmer_ACP_CA14v_Horizontal_Px15.0mm_Py10.0mm -> Potentiometers:Potentiometer_Trimmer_ACP_CA9v_Horizontal_Px10.0mm_Py5.0mm
- SW2: footprint Connector:BotaoOnOff -> Connector:BotaoOnOffMenor
Connections:
- wire segments 48 -> 51
- no-connect marks 5 -> 4
Other:
- moved on the sheet: C1
